Commit message: Initial evaluation script
As of now it computes grasp prediction from the pregenerated scenes.
Proper grasp behaviour is still to be implemented at the simulation
level

File: simulator/gripper.urdf (robot description, URDF)
Before this commit: robot myfirst, 4 links, 3 joints
Links:
- removed link palm
- added link p
- added link r
- added link world
- added link x
- added link y
- added link z
- link base_link: geometry collision box size=0.12 0.01 0.02; visual box size=0.12 0.01 0.02
Joints:
- removed joint actuator
- added joint p_joint: type revolute, parent r, child p, origin xyz=0 0 0 rpy=0 0 0, axis 0 1 0, limit lower=0 upper=6.283 effort=1000.0 velocity=0.5
- added joint r_joint: type revolute, parent z, child r, origin xyz=0 0 0 rpy=0 0 0, axis 1 0 0, limit lower=0 upper=6.283 effort=1000.0 velocity=0.5
- added joint x_joint: type prismatic, parent world, child x, origin xyz=0 0 2 rpy=0 0 0, axis 1 0 0, limit lower=-10 upper=10 effort=1000.0 velocity=0.5
- added joint y_joint: type prismatic, parent x, child y, origin xyz=0 0 0 rpy=0 0 0, axis 0 1 0, limit lower=-10 upper=10 effort=1000.0 velocity=0.5
- added joint yy_joint: type revolute, parent p, child base_link, origin xyz=0 0 0 rpy=-1.57 0 0, axis 0 -1 0, limit lower=0 upper=6.283 effort=1000.0 velocity=0.5
- added joint z_joint: type prismatic, parent y, child z, origin xyz=0 0 0 rpy=0 0 0, axis 0 0 1, limit lower=-10 upper=10 effort=1000.0 velocity=0.5
- joint left_joint: limit lower=0 upper=0.05 effort=1000.0 velocity=0.5 -> lower=0 upper=0.05 effort=1000.0 velocity=0.001; parent palm -> base_link
- joint right_joint: limit lower=-0.05 upper=0 effort=1000.0 velocity=-0.5 -> lower=-0.05 upper=0 effort=1000.0 velocity=-0.001; parent palm -> base_link

Commit message: Working grasp physics

File: simulator/gripper.urdf (robot description, URDF)
Before this commit: robot gripper, 9 links, 8 joints
Joints:
- joint left_joint: limit lower=0 upper=0.05 effort=1000.0 velocity=0.001 -> lower=0 upper=0.05 effort=1000.0
- joint p_joint: limit lower=0 upper=6.283 effort=1000.0 velocity=0.5 -> lower=0 upper=6.283 effort=1000.0 velocity=0.01
- joint r_joint: limit lower=0 upper=6.283 effort=1000.0 velocity=0.5 -> lower=0 upper=6.283 effort=1000.0 velocity=0.01
- joint right_joint: axis (none) -> -1 0 0; limit lower=-0.05 upper=0 effort=1000.0 velocity=-0.001 -> lower=0 upper=0.05 effort=1000.0
- joint x_joint: limit lower=-10 upper=10 effort=1000.0 velocity=0.5 -> lower=-10 upper=10 effort=1000.0 velocity=0.01; origin xyz=0 0 2 rpy=0 0 0 -> xyz=0 0 0 rpy=0 0 0
- joint y_joint: limit lower=-10 upper=10 effort=1000.0 velocity=0.5 -> lower=-10 upper=10 effort=1000.0 velocity=0.01
- joint z_joint: limit lower=-10 upper=10 effort=1000.0 velocity=0.5 -> lower=-10 upper=10 effort=1000.0 velocity=0.01

Commit message: Refactoring and fix gripper rotational joint limits

File: simulator/gripper.urdf (robot description, URDF)
Before this commit: robot gripper, 9 links, 8 joints
Joints:
- joint p_joint: limit lower=0 upper=6.283 effort=1000.0 velocity=0.01 -> lower=-1.58 upper=1.58 effort=1000.0 velocity=0.01
- joint r_joint: limit lower=0 upper=6.283 effort=1000.0 velocity=0.01 -> lower=-1.58 upper=1.58 effort=1000.0 velocity=0.01
- joint yy_joint: limit lower=0 upper=6.283 effort=1000.0 velocity=0.5 -> lower=-1.58 upper=1.58 effort=1000.0 velocity=0.5

Commit message: Proper video logging and obj rescaling

File: simulator/gripper.urdf (robot description, URDF)
Before this commit: robot gripper, 9 links, 8 joints
Links:
- link base_link: geometry collision box size=0.32 0.01 0.02; visual box size=0.32 0.01 0.02
Joints:
- joint left_joint: limit lower=0 upper=0.05 effort=1000.0 -> lower=0 upper=0.15 effort=1000.0
- joint right_joint: limit lower=0 upper=0.05 effort=1000.0 -> lower=0 upper=0.15 effort=1000.0
