Commit message: New scene format and improved results metadata

File: simulator/gripper_wide.urdf (robot description, URDF)
Before this commit: robot gripper, 9 links, 8 joints
Links:
- link base_link: geometry collision box size=0.32 0.01 0.06; visual box size=0.32 0.01 0.06
- link left_jaw: geometry collision box size=0.05 0.01 0.06; visual box size=0.05 0.01 0.06
- link right_jaw: geometry collision box size=0.05 0.01 0.06; visual box size=0.05 0.01 0.06
